File: viper_v1.kicad_pcb (KiCad board)
At the start: 2 copper layers, 285 x 94.6 mm, 26 parts, among them J1 AVR-ISP-6, SW1 SW_Push, SW2 SW_Push, SW3 SW_Push, SW4 SW_Push, SW5 SW_Push, U1 ATmega32U4-A, Y1 16MHz

Commit message: Added rows/columns for simple wkl layout
Added values to keys in schematic & updated meta keys

Aligned switches & diodes

Moved some footprints around to prevent overlapping.

Added PWR Flags & connected shield

Custom SKQG footprint.

Set up 15mil power netclass for +5V, VCC & GND
Parts:
- removed the D2 at (109.1, 96.8)
- removed the SW2 at (104.3, 91.3)
- added D10: D_Small, Diode_SMD:D_SOD-123, B.Cu at (221.6, 63.5)
- added D11: D_Small, Diode_SMD:D_SOD-123, B.Cu at (240.5, 63.5)
- added D12: D_Small, Diode_SMD:D_SOD-123, B.Cu at (259.7, 63.5)
- added D13: D_Small, Diode_SMD:D_SOD-123, B.Cu at (278.7, 63.5)
- added D14: D_Small, Diode_SMD:D_SOD-123, B.Cu at (307.3, 63.5)
- added D15: D_Small, Diode_SMD:D_SOD-123, B.Cu at (54.9, 82.5)
- added D16: D_Small, Diode_SMD:D_SOD-123, B.Cu at (78.7, 82.5)
- added D17: D_Small, Diode_SMD:D_SOD-123, B.Cu at (97.7, 82.5)
- added D18: D_Small, Diode_SMD:D_SOD-123, B.Cu at (116.8, 82.5)
- added D19: D_Small, Diode_SMD:D_SOD-123, B.Cu at (135.8, 82.5)
- added D20: D_Small, Diode_SMD:D_SOD-123, B.Cu at (154.9, 82.5)
- added D21: D_Small, Diode_SMD:D_SOD-123, B.Cu at (173.9, 82.5)
- added D22: D_Small, Diode_SMD:D_SOD-123, B.Cu at (193.0, 82.5)
- added D23: D_Small, Diode_SMD:D_SOD-123, B.Cu at (212.0, 82.5)
- added D24: D_Small, Diode_SMD:D_SOD-123, B.Cu at (231.1, 82.5)
- added D25: D_Small, Diode_SMD:D_SOD-123, B.Cu at (250.1, 82.5)
- added D26: D_Small, Diode_SMD:D_SOD-123, B.Cu at (269.2, 82.5)
- added D27: D_Small, Diode_SMD:D_SOD-123, B.Cu at (288.2, 82.5)
- added D28: D_Small, Diode_SMD:D_SOD-123, B.Cu at (312.0, 82.5)
- added D29: D_Small, Diode_SMD:D_SOD-123, B.Cu at (57.2, 101.6)
- added D3: D_Small, Diode_SMD:D_SOD-123, B.Cu at (88.2, 63.5)
- added D30: D_Small, Diode_SMD:D_SOD-123, B.Cu at (83.4, 101.6)
- added D31: D_Small, Diode_SMD:D_SOD-123, B.Cu at (102.5, 101.6)
- added D32: D_Small, Diode_SMD:D_SOD-123, B.Cu at (121.5, 101.6)
- added D33: D_Small, Diode_SMD:D_SOD-123, B.Cu at (140.6, 101.6)
- added D34: D_Small, Diode_SMD:D_SOD-123, B.Cu at (159.6, 101.6)
- added D35: D_Small, Diode_SMD:D_SOD-123, B.Cu at (178.6, 101.6)
- added D36: D_Small, Diode_SMD:D_SOD-123, B.Cu at (197.7, 101.6)
- added D37: D_Small, Diode_SMD:D_SOD-123, B.Cu at (216.8, 101.6)
- added D38: D_Small, Diode_SMD:D_SOD-123, B.Cu at (235.8, 101.6)
- added D39: D_Small, Diode_SMD:D_SOD-123, B.Cu at (254.9, 101.6)
- added D40: D_Small, Diode_SMD:D_SOD-123, B.Cu at (273.9, 101.6)
- added D41: D_Small, Diode_SMD:D_SOD-123, B.Cu at (304.9, 101.6)
- added D42: D_Small, Diode_SMD:D_SOD-123, B.Cu at (62.0, 120.7)
- added D43: D_Small, Diode_SMD:D_SOD-123, B.Cu at (93.0, 120.7)
- added D44: D_Small, Diode_SMD:D_SOD-123, B.Cu at (112.0, 120.7)
- added D45: D_Small, Diode_SMD:D_SOD-123, B.Cu at (131.1, 120.7)
- added D46: D_Small, Diode_SMD:D_SOD-123, B.Cu at (150.2, 120.7)
- added D47: D_Small, Diode_SMD:D_SOD-123, B.Cu at (169.1, 120.7)
- added D48: D_Small, Diode_SMD:D_SOD-123, B.Cu at (188.2, 120.7)
- added D49: D_Small, Diode_SMD:D_SOD-123, B.Cu at (207.3, 120.7)
- added D5: D_Small, Diode_SMD:D_SOD-123, B.Cu at (126.3, 63.5)
- added D50: D_Small, Diode_SMD:D_SOD-123, B.Cu at (226.3, 120.7)
- added D51: D_Small, Diode_SMD:D_SOD-123, B.Cu at (245.4, 120.7)
- added D52: D_Small, Diode_SMD:D_SOD-123, B.Cu at (264.4, 120.7)
- added D53: D_Small, Diode_SMD:D_SOD-123, B.Cu at (300.1, 120.7)
- added D54: D_Small, Diode_SMD:D_SOD-123, B.Cu at (78.6, 139.7)
- added D55: D_Small, Diode_SMD:D_SOD-123, B.Cu at (102.5, 139.7)
- added D56: D_Small, Diode_SMD:D_SOD-123, B.Cu at (183.4, 139.7)
- added D57: D_Small, Diode_SMD:D_SOD-123, B.Cu at (278.6, 139.7)
- added D58: D_Small, Diode_SMD:D_SOD-123, B.Cu at (254.9, 139.7)
- added D6: D_Small, Diode_SMD:D_SOD-123, B.Cu at (145.4, 63.5)
- added D7: D_Small, Diode_SMD:D_SOD-123, B.Cu at (154.9, 63.5)
- added D8: D_Small, Diode_SMD:D_SOD-123, B.Cu at (183.4, 63.5)
- added D9: D_Small, Diode_SMD:D_SOD-123, B.Cu at (202.5, 63.5)
- added SW10: KC_9, MX_Solderable:MX-Solderable-1U, F.Cu at (216.9, 57.9)
- added SW11: KC_0, MX_Solderable:MX-Solderable-1U, F.Cu at (235.9, 57.9)
- added SW12: KC_MINS, MX_Solderable:MX-Solderable-1U, F.Cu at (255.0, 57.9)
- added SW13: KC_EQL, MX_Solderable:MX-Solderable-1U, F.Cu at (274.0, 57.9)
- added SW14: KC_BSPC, MX_Solderable:MX-Solderable-2U, F.Cu at (302.5, 57.9)
- added SW15: KC_TAB, MX_Solderable:MX-Solderable-1.5U, F.Cu at (50.1, 77.0)
- added SW16: KC_Q, MX_Solderable:MX-Solderable-1U, F.Cu at (73.9, 77.0)
- added SW17: KC_W, MX_Solderable:MX-Solderable-1U, F.Cu at (93.0, 77.0)
- added SW18: KC_E, MX_Solderable:MX-Solderable-1U, F.Cu at (112.0, 77.0)
- added SW19: KC_R, MX_Solderable:MX-Solderable-1U, F.Cu at (131.1, 77.0)
- added SW20: KC_T, MX_Solderable:MX-Solderable-1U, F.Cu at (150.1, 77.0)
- added SW21: KC_Y, MX_Solderable:MX-Solderable-1U, F.Cu at (169.2, 77.0)
- added SW22: KC_U, MX_Solderable:MX-Solderable-1U, F.Cu at (188.2, 77.0)
- added SW23: KC_I, MX_Solderable:MX-Solderable-1U, F.Cu at (207.3, 77.0)
- added SW24: KC_O, MX_Solderable:MX-Solderable-1U, F.Cu at (226.3, 77.0)
- added SW25: KC_P, MX_Solderable:MX-Solderable-1U, F.Cu at (245.4, 77.0)
- added SW26: KC_LBRC, MX_Solderable:MX-Solderable-1U, F.Cu at (264.4, 77.0)
- added SW27: KC_RBRC, MX_Solderable:MX-Solderable-1U, F.Cu at (283.5, 77.0)
- added SW28: KC_BSLS, MX_Solderable:MX-Solderable-1.5U, F.Cu at (307.3, 77.0)
- added SW29: KC_CAPS, MX_Solderable:MX-Solderable-1.75U, F.Cu at (52.5, 96.0)
- added SW3: KC_2, MX_Solderable:MX-Solderable-1U, F.Cu at (83.5, 57.9)
- added SW30: KC_A, MX_Solderable:MX-Solderable-1U, F.Cu at (78.7, 96.0)
- added SW31: KC_S, MX_Solderable:MX-Solderable-1U, F.Cu at (97.7, 96.0)
- added SW32: KC_D, MX_Solderable:MX-Solderable-1U, F.Cu at (116.8, 96.0)
- added SW33: KC_F, MX_Solderable:MX-Solderable-1U, F.Cu at (135.8, 96.0)
- added SW34: KC_G, MX_Solderable:MX-Solderable-1U, F.Cu at (154.9, 96.0)
- added SW35: KC_H, MX_Solderable:MX-Solderable-1U, F.Cu at (173.9, 96.0)
- added SW36: KC_J, MX_Solderable:MX-Solderable-1U, F.Cu at (193.0, 96.0)
- added SW37: KC_K, MX_Solderable:MX-Solderable-1U, F.Cu at (212.0, 96.0)
- added SW38: KC_L, MX_Solderable:MX-Solderable-1U, F.Cu at (231.1, 96.0)
- added SW39: KC_SCLN, MX_Solderable:MX-Solderable-1U, F.Cu at (250.1, 96.0)
- added SW40: KC_QUOT, MX_Solderable:MX-Solderable-1U, F.Cu at (269.2, 96.0)
- added SW41: KC_ENT, MX_Solderable:MX-Solderable-2.25U-ReversedStabilizers, F.Cu at (300.1, 96.0)
- added SW42: KC_LSFT, MX_Solderable:MX-Solderable-2.25U-ReversedStabilizers, F.Cu at (57.2, 115.1)
- added SW43: KC_Z, MX_Solderable:MX-Solderable-1U, F.Cu at (88.2, 115.1)
- added SW44: KC_X, MX_Solderable:MX-Solderable-1U, F.Cu at (107.3, 115.1)
- added SW45: KC_C, MX_Solderable:MX-Solderable-1U, F.Cu at (126.3, 115.1)
- added SW46: KC_V, MX_Solderable:MX-Solderable-1U, F.Cu at (145.4, 115.1)
- added SW47: KC_B, MX_Solderable:MX-Solderable-1U, F.Cu at (164.4, 115.1)
- added SW48: KC_N, MX_Solderable:MX-Solderable-1U, F.Cu at (183.5, 115.1)
- added SW49: KC_M, MX_Solderable:MX-Solderable-1U, F.Cu at (202.5, 115.1)
- added SW50: KC_COMM, MX_Solderable:MX-Solderable-1U, F.Cu at (221.6, 115.1)
- added SW51: KC_DOT, MX_Solderable:MX-Solderable-1U, F.Cu at (240.6, 115.1)
- added SW52: KC_SLSH, MX_Solderable:MX-Solderable-1U, F.Cu at (259.7, 115.1)
- added SW53: KC_RSFT, MX_Solderable:MX-Solderable-2.75U-ReversedStabilizers, F.Cu at (295.4, 115.1)
- added SW54: KC_LEFT_GUI, MX_Solderable:MX-Solderable-1U, F.Cu at (73.8, 134.1)
- added SW55: KC_LEFT_ALT, MX_Solderable:MX-Solderable-1.5U, F.Cu at (97.7, 134.1)
- added SW56: KC_SPACE, MX_Solderable:MX-Solderable-7U-ReversedStabilizers, F.Cu at (178.7, 134.1)
- added SW57: KC_RIGHT_GUI, MX_Solderable:MX-Solderable-1U, F.Cu at (283.4, 134.1)
- added SW58: KC_RIGHT_ALT, MX_Solderable:MX-Solderable-1.5U, F.Cu at (259.6, 134.1)
- added SW59: SW_RESET, random-keyboard-parts:SKQG-1155865, B.Cu at (66.6, 93.7)
- added SW6: KC_5, MX_Solderable:MX-Solderable-1U, F.Cu at (140.7, 57.9)
- added SW7: KC_6, MX_Solderable:MX-Solderable-1U, F.Cu at (159.7, 57.9)
- added SW8: KC_7, MX_Solderable:MX-Solderable-1U, F.Cu at (178.8, 57.9)
- added SW9: KC_8, MX_Solderable:MX-Solderable-1U, F.Cu at (197.8, 57.9)
- SW1: value SW_Push -> KC_GRV
- SW2: renamed from SW3; value SW_Push -> KC_1
- SW4: value SW_Push -> KC_3
- SW5: value SW_Push -> KC_4; footprint random-keyboard-parts:SKQG-1155865 -> MX_Solderable:MX-Solderable-1U; moved to F.Cu
- moved C6 123.7 mm to (156.8, 134.9), turned to 180 degrees
- moved C5 117.5 mm to (156.8, 132.6)
- moved Y1 117.4 mm to (152.7, 133.8), turned to 0 degrees
- moved U1 115.9 mm to (139.8, 132.8), turned to 0 degrees
- moved C2 115.9 mm to (147.6, 126.2)
- moved C4 115.9 mm to (132.1, 139.6)
- moved R1 115.9 mm to (143.7, 122.9)
- moved C3 115.9 mm to (133.1, 125.2)
- moved C7 115.9 mm to (138.9, 122.9)
- moved C1 115.9 mm to (146.6, 140.5)
- moved SW5 94.4 mm to (121.6, 57.9), turned to 0 degrees
- moved J1 89.0 mm to (120.0, 133.9)
- moved D1 59.7 mm to (40.5, 63.5)
- moved R4 59.1 mm to (65.9, 101.6)
- moved R2 56.9 mm to (55.9, 60.3)
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- renumbered D3 to D2, R3 to R1, R1 to R3
Connections:
- net /D+ renamed D+
- net /D- renamed D-
- net Net-(U1-XTAL1) renamed XTAL1
- net Net-(U1-XTAL2) renamed XTAL2
- D4 pad 1: Row1 -> Row0
- SW4 pad 1: Col1 -> Col3
- SW5 pad 1: GND -> Col4
- SW5 pad 2: RST -> Net-(D5-A)
- U1 pad 1: unconnected-(U1-PE6-Pad1) -> Row0
- U1 pad 19: unconnected-(U1-PD1-Pad19) -> Col8
- U1 pad 20: unconnected-(U1-PD2-Pad20) -> Col9
- U1 pad 21: unconnected-(U1-PD3-Pad21) -> Col10
- U1 pad 22: unconnected-(U1-PD5-Pad22) -> Col11
- U1 pad 25: unconnected-(U1-PD4-Pad25) -> Col12
- U1 pad 26: unconnected-(U1-PD6-Pad26) -> Col13
- U1 pad 27: Row0 -> unconnected-(U1-PD7-Pad27)
- U1 pad 28: Col1 -> Col0
- U1 pad 29: Col0 -> Col1
- U1 pad 30: Row1 -> Col2
- U1 pad 31: unconnected-(U1-PC6-Pad31) -> Col3
- U1 pad 32: unconnected-(U1-PC7-Pad32) -> Col4
- U1 pad 36: unconnected-(U1-PF7-Pad36) -> Col6
- U1 pad 37: unconnected-(U1-PF6-Pad37) -> Col5
- U1 pad 38: unconnected-(U1-PF5-Pad38) -> Row1
- U1 pad 39: unconnected-(U1-PF4-Pad39) -> Row4
- U1 pad 40: unconnected-(U1-PF1-Pad40) -> Row3
- U1 pad 41: unconnected-(U1-PF0-Pad41) -> Row2
- U1 pad 8: unconnected-(U1-PB0-Pad8) -> Col7
- USB1 pad 6: unconnected-(USB1-SHIELD-Pad6) -> GND

Commit message: Moved footprints to 0,0
Added better mounting holes

Testing different usb miniB footprints & replaced mounting holes.

Added another decoupling cap.

Reannotated parts

Centered diodes under switches where possible

Changed PCB edges around USB connector & added (optional) rounded corners.

45deg corners

Swapped rows/columns

Adding additional switch footprints.
Parts:
- removed the SW3 at (83.5, 57.9)
- removed USB1: Molex-0548190589, random-keyboard-parts:Molex-0548190589
- removed viper-v1-outline: viper_v1_outline, outline:viper_v1_outline
- added C7: 0.1uF, Capacitor_SMD:C_0805_2012Metric, B.Cu at (110.5, 82.9)
- added J1: USB_B_Mini, local:USB_miniB_hirose_5ST_hand, B.Cu at (9.00, -6.36)
- added S1: Screw_Terminal_01x01, local:10x5_7x2.5mm, F.Cu at (121.0, 8.05)
- added S2: Screw_Terminal_01x01, local:5.5_5x2.5mm, F.Cu at (250.8, 18.7)
- added S3: Screw_Terminal_01x01, local:5.5_5x2.5mm, F.Cu at (16.0, 18.7)
- added S4: Screw_Terminal_01x01, local:5.5_5x2.5mm, F.Cu at (119.0, 37.8)
- added S5: Screw_Terminal_01x01, local:10x5_7x2.5mm, F.Cu at (275.8, 47.3)
- added S6: Screw_Terminal_01x01, local:10x5_7x2.5mm, F.Cu at (-9.20, 47.3)
- added S7: Screw_Terminal_01x01, local:5.5_5x2.5mm, F.Cu at (181.3, 76.0)
- added S8: Screw_Terminal_01x01, local:10x5_7x2.5mm, F.Cu at (223.8, 85.4)
- added S9: Screw_Terminal_01x01, local:10x5_7x2.5mm, F.Cu at (42.8, 85.4)
- added SW4: KC_2, MX_Solderable:MX-Solderable-1U, F.Cu at (38.1, 0.00)
- moved R1 154.1 mm to (19.8, 31.2)
- moved C3 87.8 mm to (96.5, 68.4), turned to 180 degrees
- moved D46 81.5 mm to (93.7, 61.9), turned to 90 degrees
- moved D14 78.6 mm to (251.6, 7.94)
- moved D54 75.4 mm to (28.6, 83.3)
- moved D55 75.4 mm to (52.4, 83.3)
- moved D56 75.4 mm to (133.3, 83.3)
- moved D2 74.9 mm to (19.1, 7.94)
- moved D37 74.9 mm to (166.6, 46.0)
- moved D39 74.9 mm to (204.7, 46.0)
- moved D16 74.9 mm to (28.5, 27.0)
- moved D32 74.9 mm to (71.4, 46.0)
- moved D10 74.8 mm to (171.4, 7.94)
- moved D12 74.8 mm to (209.6, 7.94)
- moved D19 74.8 mm to (85.7, 27.0)
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- renumbered C5 to C1, C6 to C2, C1 to C3, C2 to C4, C3 to C5, C4 to C6, C7 to C8, J1 to J2, SW59 to SW1, SW9 to SW10, SW10 to SW11, SW11 to SW12, SW12 to SW13, SW13 to SW14, SW14 to SW15, SW15 to SW16, SW16 to SW17, SW17 to SW18, SW18 to SW19, SW1 to SW2, SW19 to SW20, SW20 to SW21, SW21 to SW22, SW22 to SW23, SW23 to SW24, SW24 to SW25, SW25 to SW26, SW26 to SW27, SW27 to SW28, SW28 to SW29, SW2 to SW3, SW29 to SW30, SW30 to SW31, SW31 to SW32, SW32 to SW33, SW33 to SW34, SW34 to SW35, SW35 to SW36, SW36 to SW37, SW37 to SW38, SW38 to SW39, SW39 to SW40, SW40 to SW41, SW41 to SW42, SW42 to SW43, SW43 to SW44, SW44 to SW45, SW45 to SW46, SW46 to SW47, SW47 to SW48, SW48 to SW49, SW4 to SW5, SW49 to SW50, SW50 to SW51, SW51 to SW52, SW52 to SW53, SW53 to SW54, SW54 to SW55, SW55 to SW56, SW56 to SW57, SW57 to SW58, SW58 to SW59, SW5 to SW6, SW6 to SW7, SW7 to SW8, SW8 to SW9
Connections:
- SW10 pad 1: Col8 -> Net-(D9-A)
- SW10 pad 2: Net-(D9-A) -> Col8
- SW11 pad 1: Col9 -> Net-(D10-A)
- SW11 pad 2: Net-(D10-A) -> Col9
- SW12 pad 1: Col10 -> Net-(D11-A)
- SW12 pad 2: Net-(D11-A) -> Col10
- SW13 pad 1: Col11 -> Net-(D12-A)
- SW13 pad 2: Net-(D12-A) -> Col11
- SW14 pad 1: Col12 -> Net-(D13-A)
- SW14 pad 2: Net-(D13-A) -> Col12
- SW15 pad 1: Col13 -> Net-(D14-A)
- SW15 pad 2: Net-(D14-A) -> Col13
- SW16 pad 1: Col0 -> Net-(D15-A)
- SW16 pad 2: Net-(D15-A) -> Col0
- SW17 pad 1: Col1 -> Net-(D16-A)
- SW17 pad 2: Net-(D16-A) -> Col1
- SW18 pad 1: Col2 -> Net-(D17-A)
- SW18 pad 2: Net-(D17-A) -> Col2
- SW19 pad 1: Col3 -> Net-(D18-A)
- SW19 pad 2: Net-(D18-A) -> Col3
- SW2 pad 1: Col0 -> Net-(D1-A)
- SW2 pad 2: Net-(D1-A) -> Col0
- SW20 pad 1: Col4 -> Net-(D19-A)
- SW20 pad 2: Net-(D19-A) -> Col4
- SW21 pad 1: Col5 -> Net-(D20-A)
- SW21 pad 2: Net-(D20-A) -> Col5
- SW22 pad 1: Col6 -> Net-(D21-A)
- SW22 pad 2: Net-(D21-A) -> Col6
- SW23 pad 1: Col7 -> Net-(D22-A)
- SW23 pad 2: Net-(D22-A) -> Col7
- SW24 pad 1: Col8 -> Net-(D23-A)
- SW24 pad 2: Net-(D23-A) -> Col8
- SW25 pad 1: Col9 -> Net-(D24-A)
- SW25 pad 2: Net-(D24-A) -> Col9
- SW26 pad 1: Col10 -> Net-(D25-A)
- SW26 pad 2: Net-(D25-A) -> Col10
- SW27 pad 1: Col11 -> Net-(D26-A)
- SW27 pad 2: Net-(D26-A) -> Col11
- SW28 pad 1: Col12 -> Net-(D27-A)
- SW28 pad 2: Net-(D27-A) -> Col12
- SW29 pad 1: Col13 -> Net-(D28-A)
- SW29 pad 2: Net-(D28-A) -> Col13
- SW3 pad 1: Col1 -> Net-(D2-A)
- SW3 pad 2: Net-(D2-A) -> Col1
- SW30 pad 1: Col0 -> Net-(D29-A)
- SW30 pad 2: Net-(D29-A) -> Col0
- SW31 pad 1: Col1 -> Net-(D30-A)
- SW31 pad 2: Net-(D30-A) -> Col1
- SW32 pad 1: Col2 -> Net-(D31-A)
- SW32 pad 2: Net-(D31-A) -> Col2
- SW33 pad 1: Col3 -> Net-(D32-A)
- SW33 pad 2: Net-(D32-A) -> Col3
- SW34 pad 1: Col4 -> Net-(D33-A)
- SW34 pad 2: Net-(D33-A) -> Col4
- SW35 pad 1: Col5 -> Net-(D34-A)
- SW35 pad 2: Net-(D34-A) -> Col5
- SW36 pad 1: Col6 -> Net-(D35-A)
- SW36 pad 2: Net-(D35-A) -> Col6
- SW37 pad 1: Col7 -> Net-(D36-A)
- SW37 pad 2: Net-(D36-A) -> Col7
- SW38 pad 1: Col8 -> Net-(D37-A)
- SW38 pad 2: Net-(D37-A) -> Col8
- SW39 pad 1: Col9 -> Net-(D38-A)
- SW39 pad 2: Net-(D38-A) -> Col9
- SW40 pad 1: Col10 -> Net-(D39-A)
- SW40 pad 2: Net-(D39-A) -> Col10
- SW41 pad 1: Col11 -> Net-(D40-A)
- SW41 pad 2: Net-(D40-A) -> Col11
- SW42 pad 1: Col13 -> Net-(D41-A)
- SW42 pad 2: Net-(D41-A) -> Col13
- SW43 pad 1: Col0 -> Net-(D42-A)
- SW43 pad 2: Net-(D42-A) -> Col0
- SW44 pad 1: Col2 -> Net-(D43-A)
- SW44 pad 2: Net-(D43-A) -> Col2
- SW45 pad 1: Col3 -> Net-(D44-A)
- SW45 pad 2: Net-(D44-A) -> Col3
- SW46 pad 1: Col4 -> Net-(D45-A)
- SW46 pad 2: Net-(D45-A) -> Col4
- SW47 pad 1: Col5 -> Net-(D46-A)
- SW47 pad 2: Net-(D46-A) -> Col5
- SW48 pad 1: Col6 -> Net-(D47-A)
- SW48 pad 2: Net-(D47-A) -> Col6
- SW49 pad 1: Col7 -> Net-(D48-A)
- SW49 pad 2: Net-(D48-A) -> Col7
- SW5 pad 1: Col3 -> Net-(D4-A)
- SW5 pad 2: Net-(D4-A) -> Col3
- SW50 pad 1: Col8 -> Net-(D49-A)
- SW50 pad 2: Net-(D49-A) -> Col8
- SW51 pad 1: Col9 -> Net-(D50-A)
- SW51 pad 2: Net-(D50-A) -> Col9
- SW52 pad 1: Col10 -> Net-(D51-A)
- SW52 pad 2: Net-(D51-A) -> Col10
- SW53 pad 1: Col11 -> Net-(D52-A)
- SW53 pad 2: Net-(D52-A) -> Col11
- SW54 pad 1: Col13 -> Net-(D53-A)
- SW54 pad 2: Net-(D53-A) -> Col13
- SW55 pad 1: Col1 -> Net-(D54-A)
- SW55 pad 2: Net-(D54-A) -> Col1
- SW56 pad 1: Col2 -> Net-(D55-A)
- SW56 pad 2: Net-(D55-A) -> Col2
- SW57 pad 1: Col6 -> Net-(D56-A)
- SW57 pad 2: Net-(D56-A) -> Col6
- SW58 pad 1: Col10 -> Net-(D57-A)
- SW58 pad 2: Net-(D57-A) -> Col10
- SW59 pad 1: Col11 -> Net-(D58-A)
- SW59 pad 2: Net-(D58-A) -> Col11
- SW6 pad 1: Col4 -> Net-(D5-A)
- SW6 pad 2: Net-(D5-A) -> Col4
- SW7 pad 1: Col5 -> Net-(D6-A)
- SW7 pad 2: Net-(D6-A) -> Col5
- SW8 pad 1: Col6 -> Net-(D7-A)
- SW8 pad 2: Net-(D7-A) -> Col6
- SW9 pad 1: Col7 -> Net-(D8-A)
- SW9 pad 2: Net-(D8-A) -> Col7
Routing:
- net Row1: track 0.00 -> 268.5 mm, vias 0 -> 2
- net Row0: track 0.00 -> 268.4 mm, vias 0 -> 2
- net Row2: track 0.00 -> 245.2 mm
- net Row4: track 0.00 -> 223.3 mm, vias 0 -> 2
- net Row3: track 0.00 -> 179.0 mm
- net D-: track 0.00 -> 153.8 mm
- net D+: track 0.00 -> 153.8 mm
- net Col10: track 0.00 -> 117.8 mm
- net Col6: track 0.00 -> 93.3 mm
- net Col2: track 0.00 -> 90.0 mm
- net Col11: track 0.00 -> 86.7 mm, vias 0 -> 1
- net Col1: track 0.00 -> 84.1 mm
- net Col7: track 0.00 -> 67.0 mm
- net Col9: track 0.00 -> 67.0 mm
- net Col4: track 0.00 -> 67.0 mm
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Other:
- board size 285 x 94.6 mm -> 285 x 97.8 mm

Commit message: Placed new footprints for iso enter, short shifts, stepped caps, fn & 2 more iso switches.
Added USBLC6-2SC6 for ESD protection
Parts:
- added D15: D_Small, Diode_SMD:D_SOD-123, B.Cu at (236.5, 1.40)
- added D42: D_Small, Diode_SMD:D_SOD-123, B.Cu at (32.5, 57.1)
- added D45: D_Small, Diode_SMD:D_SOD-123, B.Cu at (234.2, 38.8)
- added D56: D_Small, Diode_SMD:D_SOD-123, B.Cu at (230.2, 56.3)
- added SW16: KC_BSPC1, MX_Solderable:MX-Solderable-1U, F.Cu at (247.7, 0.00)
- added SW17: KC_DEL, MX_Solderable:MX-Solderable-1U, F.Cu at (266.7, 0.00)
- added SW44: KC_ISO_1, MX_Solderable:MX-Solderable-1U, F.Cu at (23.8, 57.1)
- added SW46: KC_CAPS, MX_Solderable:MX-Solderable-1.75U, F.Cu at (7.14, 38.1)
- added SW47: KC_ENT, MX_Solderable:MX-Solderable-2.25U-ReversedStabilizers, F.Cu at (254.8, 38.1)
- added SW48: KC_LSHIFT_SHORT, MX_Solderable:MX-Solderable-1.25U, F.Cu at (2.38, 57.1)
- added SW49: KC_ISO_2, MX_Solderable:MX-Solderable-1U, F.Cu at (242.9, 38.1)
- added SW60: KC_RSFT_SHORT, MX_Solderable:MX-Solderable-1.75U, F.Cu at (240.5, 57.1)
- added SW63: KC_RSFT, MX_Solderable:MX-Solderable-2.75U-ReversedStabilizers, F.Cu at (250.0, 57.1)
- SW32: renamed from SW30; value KC_CAPS -> KC_CAPS_STEP; footprint MX_Solderable:MX-Solderable-1.75U -> MX_Solderable:MX-Solderable-1.25U
- SW45: renamed from SW42; value KC_ENT -> KC_ENT_ISO; footprint MX_Solderable:MX-Solderable-2.25U-ReversedStabilizers -> MX_Solderable:MX-Solderable-2U-Vertical
- SW61: renamed from SW54; value KC_RSFT -> KC_FN; footprint MX_Solderable:MX-Solderable-2.75U-ReversedStabilizers -> MX_Solderable:MX-Solderable-1U
- moved D29 32.9 mm to (229.7, 20.4), turned to 90 degrees
- moved D1 27.7 mm to (26.9, 1.40), turned to 90 degrees
- moved SW61 16.7 mm to (266.7, 57.1)
- moved D8 14.7 mm to (124.8, 1.40), turned to 90 degrees
- moved D14 14.1 mm to (239.2, 1.40), turned to 90 degrees
- moved SW45 13.5 mm to (264.4, 28.6)
- moved D28 12.8 mm to (227.1, 20.4), turned to 90 degrees
- moved D2 12.4 mm to (29.6, 1.40), turned to 90 degrees
- moved D13 10.8 mm to (220.1, 1.40), turned to 90 degrees
- moved D12 10.7 mm to (201.0, 1.40), turned to 90 degrees
- moved D9 10.7 mm to (143.9, 1.40), turned to 90 degrees
- moved D4 10.7 mm to (48.6, 1.40), turned to 90 degrees
- moved D5 10.7 mm to (67.7, 1.40), turned to 90 degrees
- moved D6 10.7 mm to (86.7, 1.40), turned to 90 degrees
- moved D10 10.7 mm to (162.9, 1.40), turned to 90 degrees
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- renumbered D15 to D16, D16 to D17, D17 to D18, D18 to D19, D19 to D20, D20 to D21, D21 to D22, D22 to D23, D23 to D24, D24 to D25, D25 to D26, D26 to D27, D27 to D28, D28 to D29, D29 to D30, D30 to D31, D31 to D32, D32 to D33, D33 to D34, D34 to D35, D35 to D36, D36 to D37, D37 to D38, D38 to D39, D39 to D40, D40 to D41, D41 to D43, D42 to D44, D43 to D46, D44 to D47, D45 to D48, D46 to D49, D47 to D50, D48 to D51, D49 to D52, D50 to D53, D51 to D54, D52 to D55, D53 to D57, D54 to D58, D55 to D59, D56 to D60, D57 to D61, D58 to D62, SW16 to SW18, SW17 to SW19, SW18 to SW20, SW19 to SW21, SW20 to SW22, SW21 to SW23, SW22 to SW24, SW23 to SW25, SW24 to SW26, SW25 to SW27, SW26 to SW28, SW27 to SW29, SW28 to SW30, SW29 to SW31, SW31 to SW33, SW32 to SW34, SW33 to SW35, SW34 to SW36, SW35 to SW37, SW36 to SW38, SW37 to SW39, SW38 to SW40, SW39 to SW41, SW40 to SW42, SW41 to SW43, SW44 to SW50, SW45 to SW51, SW46 to SW52, SW47 to SW53, SW48 to SW54, SW49 to SW55, SW50 to SW56, SW51 to SW57, SW52 to SW58, SW53 to SW59, SW43 to SW62, SW55 to SW64, SW56 to SW65, SW57 to SW66, SW58 to SW67, SW59 to SW68
Connections:
- D44 pad 2: Net-(D42-A) -> Net-(D44-A)
- SW62 pad 1: Net-(D42-A) -> Row3
- U1 pad 12: unconnected-(U1-PB7-Pad12) -> Col14
Routing:
- net Row1: track 268.5 -> 0.00 mm, vias 2 -> 0
- net Row0: track 268.4 -> 0.00 mm, vias 2 -> 0
- net Row2: track 245.2 -> 0.00 mm
- net Row4: track 223.3 -> 0.00 mm, vias 2 -> 0
- net Row3: track 179.0 -> 0.00 mm
- net D-: track 153.8 -> 0.00 mm
- net D+: track 153.8 -> 0.00 mm
- net Col10: track 117.8 -> 0.00 mm
- net Col6: track 93.3 -> 0.00 mm
- net Col2: track 90.0 -> 0.00 mm
- net Col11: track 86.7 -> 0.00 mm, vias 1 -> 0
- net Col1: track 84.1 -> 0.00 mm
- net Col7: track 67.0 -> 0.00 mm
- net Col9: track 67.0 -> 0.00 mm
- net Col4: track 67.0 -> 0.00 mm
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Other:
- outline, holes or cut-outs redrawn

Commit message: Fixed broken cols for stacked keys & added HRO-U-M-M5DD-W-1.kicad_mod from mymakercorner/Phoenix_Project_No1
Set wider track width for power & default.

Moved parts around usb connector around

Started wiring usb.

Added GND zones
Parts:
- added U2: USBLC6-2SC6, Package_TO_SOT_SMD:SOT-23-6, B.Cu at (9.53, 2.98)
- BUT1: renamed from SW1; value SW_RESET -> BUT_RESET; footprint random-keyboard-parts:SKQG-1155865 -> Button_Switch_SMD:SW_SPST_TL3342
- F1: footprint Fuse:Fuse_1206_3216Metric -> Fuse:Fuse_0805_2012Metric
- J1: footprint local:USB_miniB_hirose_5ST_hand -> local:HRO-U-M-M5DD-W-1
- J2: moved to B.Cu
- SW67: value KC_RIGHT_GUI -> KC_RIGHT_ALT; footprint MX_Solderable:MX-Solderable-1U -> MX_Solderable:MX-Solderable-1.5U
- SW68: value KC_RIGHT_ALT -> KC_RIGHT_GUI; footprint MX_Solderable:MX-Solderable-1.5U -> MX_Solderable:MX-Solderable-1U
- moved SW46 219.9 mm to (242.9, 38.1)
- moved SW51 219.9 mm to (23.8, 57.1)
- moved D42 203.4 mm to (235.1, 39.3)
- moved D45 200.0 mm to (35.1, 58.3)
- moved R2 111.7 mm to (8.33, 7.14)
- moved R3 107.8 mm to (10.7, 7.14)
- moved R1 98.5 mm to (107.6, 75.8), turned to 0 degrees
- moved C1 39.8 mm to (83.2, 66.9), turned to 0 degrees
- moved C2 39.2 mm to (83.2, 74.0), turned to 0 degrees
- moved Y1 35.4 mm to (83.2, 70.5), turned to -90 degrees
- moved C5 32.2 mm to (83.2, 62.1), turned to 180 degrees
- moved C4 26.9 mm to (83.2, 76.4)
- moved J2 24.0 mm to (107.6, 80.6), turned to -90 degrees
- moved SW67 23.8 mm to (214.3, 76.2)
- moved SW68 23.8 mm to (238.1, 76.2)
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- renumbered SW16 to SW15, SW15 to SW16, SW45 to SW33, SW46 to SW34, SW33 to SW35, SW34 to SW36, SW35 to SW37, SW36 to SW38, SW37 to SW39, SW38 to SW40, SW39 to SW41, SW40 to SW42, SW41 to SW43, SW42 to SW44, SW43 to SW45, SW44 to SW46, SW60 to SW49, SW62 to SW50, SW49 to SW51, SW50 to SW52, SW51 to SW53, SW52 to SW54, SW53 to SW55, SW54 to SW56, SW55 to SW57, SW56 to SW58, SW57 to SW59, SW58 to SW60, SW59 to SW61, SW63 to SW62, SW61 to SW63
Connections:
- C3 pad 1: +5V -> VCC
- C4 pad 1: +5V -> VCC
- C5 pad 1: +5V -> VCC
- C6 pad 1: +5V -> VCC
- C7 pad 1: +5V -> VCC
- F1 pad 1: VCC -> VBUS
- F1 pad 2: +5V -> VCC
- J1 pad 1: VCC -> VBUS
- J1 pad 2: D- -> /D-
- J1 pad 3: D+ -> /D+
- J2 pad 2: +5V -> VCC
- R1 pad 2: +5V -> VCC
- R2 pad 1: D+ -> Net-(R2-Pad1)
- R3 pad 1: D- -> Net-(R3-Pad1)
- SW15 pad 1: Net-(D15-A) -> Net-(D14-A)
- SW15 pad 2: Col14 -> Col13
- SW16 pad 1: Net-(D14-A) -> Net-(D15-A)
- SW16 pad 2: Col13 -> Col14
- SW19 pad 1: Net-(D17-A) -> Col1
- SW19 pad 2: Col1 -> Net-(D17-A)
- SW2 pad 1: Net-(D1-A) -> Col0
- SW2 pad 2: Col0 -> Net-(D1-A)
- SW3 pad 1: Net-(D2-A) -> Col1
- SW3 pad 2: Col1 -> Net-(D2-A)
- SW32 pad 1: Net-(D30-A) -> Col0
- SW32 pad 2: Col0 -> Net-(D30-A)
- SW34 pad 1: Row2 -> Col0
- SW34 pad 2: Col0 -> Net-(D30-A)
- SW35 pad 1: Net-(D31-A) -> Col1
- SW35 pad 2: Col1 -> Net-(D31-A)
- SW4 pad 1: Net-(D3-A) -> Col2
- SW4 pad 2: Col2 -> Net-(D3-A)
- SW47 pad 2: Row2 -> Net-(D43-A)
- SW48 pad 1: Net-(D44-A) -> Col0
- SW48 pad 2: Col0 -> Net-(D44-A)
- SW50 pad 1: Row3 -> Col0
- SW50 pad 2: Col0 -> Net-(D44-A)
- SW51 pad 1: Net-(D45-A) -> Col1
- SW51 pad 2: Col1 -> Net-(D45-A)
- SW52 pad 1: Net-(D46-A) -> Col2
- SW52 pad 2: Col2 -> Net-(D46-A)
- SW62 pad 1: Col12 -> Net-(D56-A)
- SW62 pad 2: Row3 -> Col12
- SW65 pad 1: Net-(D59-A) -> Col2
- SW65 pad 2: Col2 -> Net-(D59-A)
- SW66 pad 1: Net-(D60-A) -> Col6
- SW66 pad 2: Col6 -> Net-(D60-A)
- SW67 pad 1: Net-(D61-A) -> Col10
- SW67 pad 2: Col10 -> Net-(D61-A)
- U1 pad 1: Row0 -> Row4
- U1 pad 12: Col14 -> unconnected-(U1-PB7-Pad12)
- U1 pad 14: +5V -> VCC
- U1 pad 18: unconnected-(U1-PD0-Pad18) -> Col2
- U1 pad 19: Col8 -> Col1
- U1 pad 2: +5V -> VCC
- U1 pad 20: Col9 -> Col0
- U1 pad 21: Col10 -> Col3
- U1 pad 22: Col11 -> Col4
- U1 pad 24: +5V -> VCC
- U1 pad 25: Col12 -> Row3
- U1 pad 26: Col13 -> Row2
- U1 pad 27: unconnected-(U1-PD7-Pad27) -> Row1
- U1 pad 28: Col0 -> Row0
- U1 pad 29: Col1 -> Col5
- U1 pad 30: Col2 -> Col7
- U1 pad 31: Col3 -> Col8
- U1 pad 32: Col4 -> Col9
- U1 pad 34: +5V -> VCC
- U1 pad 36: Col6 -> Col14
- U1 pad 37: Col5 -> Col13
- U1 pad 38: Row1 -> Col12
- U1 pad 39: Row4 -> Col11
- U1 pad 40: Row3 -> Col10
- U1 pad 41: Row2 -> Col6
- U1 pad 44: +5V -> VCC
- U1 pad 7: +5V -> VCC
- U1 pad 8: Col7 -> unconnected-(U1-PB0-Pad8)
Routing:
- net VCC: track 0.00 -> 242.4 mm, vias 0 -> 2
- net Net-(U1-D+): track 0.00 -> 161.6 mm, vias 0 -> 2
- net Net-(U1-D-): track 0.00 -> 159.7 mm, vias 0 -> 2
- net RST: track 0.00 -> 113.7 mm, vias 0 -> 2
- net GND: track 0.00 -> 28.1 mm
- net VBUS: track 0.00 -> 14.9 mm
- net XTAL2: track 0.00 -> 11.6 mm
- net XTAL1: track 0.00 -> 9.52 mm
- net /D-: track 0.00 -> 6.48 mm, vias 0 -> 2
- net /D+: track 0.00 -> 4.92 mm
- net Net-(R2-Pad1): track 0.00 -> 2.22 mm
- net Net-(R3-Pad1): track 0.00 -> 2.22 mm
- added copper zone on B.Cu, net GND
- added copper zone on F.Cu, net GND
Other:
- board size 285 x 97.8 mm -> 285 x 94.6 mm

Commit message: Swapped ISP header & xtal footprint & connected all ratsnests
aligned vias

Renamed some screws & removed net labels
Parts:
- BUT1: value BUT_RESET -> BUT_RST
- D1, D10, D11, D12, D13, D14, D15, D16, D17, D18, D19, D2, D20, D21, D22, D23, D24, D25, D26, D27, D28, D29, D3, D30, D31, D32, D33, D34, D35, D36, D37, D38, D39, D4, D40, D41, D42, D43, D44, D45, D46, D47, D48, D49, D5, D50, D51, D52, D53, D54, D55, D56, D57, D58, D59, D6, D60, D61, D62, D7, D8, D9: footprint Diode_SMD:D_SOD-123 -> Diode_SMD:D_0805_2012Metric
- J2: value AVR-ISP-6 -> ISP; footprint random-keyboard-parts:Reset_Pretty-Mask -> local:isp_standard
- S1: value Screw_Terminal_01x01 -> Screw; footprint local:10x5_7x2.5mm -> local:5.5_5x2.5mm
- S2, S3, S4, S7: value Screw_Terminal_01x01 -> Screw
- S5, S6, S8, S9: value Screw_Terminal_01x01 -> Tofu Screw
- Y1: footprint Crystal:Crystal_SMD_3225-4Pin_3.2x2.5mm -> local:crystal_FA238-TSX3225
- moved D28 3.61 mm to (230.4, 20.8)
- moved D29 3.61 mm to (226.8, 20.8)
- moved C5 1.19 mm to (84.3, 62.1)
- moved D30 0.71 mm to (14.9, 40.0)
- moved D31 0.71 mm to (41.1, 40.0)
- moved D32 0.71 mm to (44.6, 40.0)
- moved D33 0.71 mm to (63.7, 40.0)
- moved D34 0.71 mm to (82.7, 40.0)
- moved D35 0.71 mm to (101.8, 40.0)
- moved D36 0.71 mm to (136.3, 40.0)
- moved D37 0.71 mm to (139.9, 40.0)
- moved D38 0.71 mm to (158.9, 40.0)
- moved D39 0.71 mm to (178.0, 40.0)
- moved D40 0.71 mm to (197.0, 40.0)
- moved D41 0.71 mm to (216.1, 40.0)
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Connections:
- net /D+ renamed D+
- net /D- renamed D-
- SW40 pad 1: Net-(D36-A) -> Col6
- SW40 pad 2: Col6 -> Net-(D36-A)
- SW65 pad 1: Col2 -> Net-(D59-A)
- SW65 pad 2: Net-(D59-A) -> Col2
- Y1 pad 2: GND -> XTAL2
- Y1 pad 3: XTAL2 -> GND
Routing:
- net Row0: track 0.00 -> 288.4 mm, vias 0 -> 2
- net Row1: track 0.00 -> 283.6 mm, vias 0 -> 2
- net Row2: track 0.00 -> 279.8 mm, vias 0 -> 2
- net Col13: track 0.00 -> 264.7 mm
- net Col14: track 0.00 -> 252.4 mm, vias 0 -> 2
- net Col12: track 0.00 -> 242.6 mm, vias 0 -> 1
- net Row3: track 0.00 -> 232.8 mm
- net Col11: track 0.00 -> 230.4 mm, vias 0 -> 1
- net Col10: track 0.00 -> 201.2 mm, vias 0 -> 1
- net Row4: track 0.00 -> 197.3 mm, vias 0 -> 3
- net Col0: track 0.00 -> 174.4 mm, vias 0 -> 1
- net Col9: track 0.00 -> 160.1 mm, vias 0 -> 1
- net Col1: track 0.00 -> 158.1 mm, vias 0 -> 1
- net Col2: track 0.00 -> 150.5 mm
- net Col8: track 0.00 -> 142.1 mm, vias 0 -> 1
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Other:
- outline, holes or cut-outs redrawn
