File: viper_v1.kicad_pcb (KiCad board)
At the start: 2 copper layers, 285 x 94.6 mm, 157 parts, among them J1 USB_B_Mini, J2 ISP, SW10 KC_8, SW11 KC_9, SW12 KC_0, SW13 KC_MINS, SW14 KC_EQL, SW15 KC_BSPC1, SW16 KC_BSPC, SW17 KC_DEL, SW18 KC_TAB, SW19 KC_Q, SW2 KC_GRV, SW20 KC_W, SW21 KC_E, SW22 KC_R, SW23 KC_T, SW24 KC_Y, SW25 KC_U, SW26 KC_I, SW27 KC_O, SW28 KC_P, SW29 KC_LBRC, SW3 KC_1, SW30 KC_RBRC, SW31 KC_BSLS, SW32 KC_CAPS_STEP, SW33 KC_ENT_ISO, SW34 KC_CAPS, SW35 KC_A, SW36 KC_S, SW37 KC_D, SW38 KC_F, SW39 KC_G, SW4 KC_2, SW40 KC_H, SW41 KC_J, SW42 KC_K, SW43 KC_L, SW44 KC_SCLN, SW45 KC_QUOT, SW46 KC_ISO_1, SW47 KC_ENT, SW48 KC_LSHIFT_SHORT, SW49 KC_RSFT_SHORT, SW5 KC_3, SW50 KC_LSFT, SW51 KC_ISO_2, SW52 KC_Z, SW53 KC_X, SW54 KC_C, SW55 KC_V, SW56 KC_B, SW57 KC_N, SW58 KC_M, SW59 KC_COMM, SW6 KC_4, SW60 KC_DOT, SW61 KC_SLSH, SW62 KC_RSFT, SW63 KC_FN, SW64 KC_LEFT_GUI, SW65 KC_LEFT_ALT, SW66 KC_SPACE, SW67 KC_RIGHT_ALT, SW68 KC_RIGHT_GUI, SW7 KC_5, SW8 KC_6, SW9 KC_7, U1 ATmega32U4-A, U2 USBLC6-2SC6, Y1 16MHz

Commit message: Added default 60 measurements on user comment 4, viper measurements on user comment 3
Moved all parts from 0,0 to 25,25
Parts:
- moved D14 35.4 mm to (264.9, 26.8)
- moved D15 35.4 mm to (261.3, 26.8)
- moved S2 35.4 mm to (275.9, 43.7)
- moved SW49 35.4 mm to (265.5, 82.2)
- moved D47 35.4 mm to (79.2, 84.1)
- moved D4 35.4 mm to (74.4, 26.8)
- moved D45 35.4 mm to (60.1, 84.1)
- moved D46 35.4 mm to (75.6, 84.1)
- moved D48 35.4 mm to (98.2, 84.1)
- moved D49 35.4 mm to (117.3, 84.1)
- moved D50 35.4 mm to (136.3, 84.1)
- moved D51 35.4 mm to (155.4, 84.1)
- moved D52 35.4 mm to (174.4, 84.1)
- moved D53 35.4 mm to (193.5, 84.1)
- moved D54 35.4 mm to (212.5, 84.1)
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Other:
- outline, holes or cut-outs redrawn
