File: keyboard/keyboard.kicad_pcb (KiCad board)
At the start: 2 copper layers, 295.9 x 105.4 mm, 138 parts, among them SW1 SW_Push, SW10 SW_Push, SW11 SW_Push, SW12 SW_Push, SW13 SW_Push, SW14 SW_Push, SW15 SW_Push, SW16 SW_Push, SW17 SW_Push, SW18 SW_Push, SW19 SW_Push, SW2 SW_Push, SW20 SW_Push, SW21 SW_Push, SW22 SW_Push, SW23 SW_Push, SW24 SW_Push, SW25 SW_Push, SW26 SW_Push, SW27 SW_Push, SW28 SW_Push, SW29 SW_Push, SW3 SW_Push, SW30 SW_Push, SW31 SW_Push, SW32 SW_Push, SW33 SW_Push, SW34 SW_Push, SW35 SW_Push, SW36 SW_Push, SW37 SW_Push, SW38 SW_Push, SW39 SW_Push, SW4 SW_Push, SW40 SW_Push, SW41 SW_Push, SW42 SW_Push, SW43 SW_Push, SW44 SW_Push, SW45 SW_Push, SW46 SW_Push, SW47 SW_Push, SW48 SW_Push, SW49 SW_Push, SW5 SW_Push, SW50 SW_Push, SW51 SW_Push, SW52 SW_Push, SW53 SW_Push, SW54 SW_Push, SW55 SW_Push, SW56 SW_Push, SW57 SW_Push, SW58 SW_Push, SW59 SW_Push, SW6 SW_Push, SW60 SW_Push, SW61 SW_Push, SW62 SW_Push, SW63 SW_Push, SW64 SW_Push, SW65 SW_Push, SW66 SW_Push, SW7 SW_Push, SW8 SW_Push, SW9 SW_Push

Commit message: Replaced edge cuts with viper footprint
Aligned outline with switch footprints.
Parts:
- added viper_v1: viper_v1_outline, local:viper_v1_outline, F.Cu at (0.00, 0.00)
- moved D13 90.8 mm to (242.9, 13.2)
- moved D14 90.8 mm to (271.5, 13.2)
- moved D15 90.8 mm to (261.9, 13.2)
- moved D18 90.8 mm to (42.9, 32.2)
- moved D19 90.8 mm to (61.9, 32.2)
- moved D21 90.8 mm to (100.0, 32.2)
- moved D23 90.8 mm to (138.1, 32.2)
- moved D24 90.8 mm to (157.2, 32.2)
- moved D26 90.8 mm to (195.3, 32.2)
- moved D27 90.8 mm to (214.3, 32.2)
- moved D3 90.8 mm to (52.4, 13.2)
- moved D30 90.8 mm to (276.2, 32.2)
- moved D34 90.8 mm to (85.7, 51.3)
- moved D36 90.8 mm to (123.8, 51.3)
- moved D38 90.8 mm to (161.9, 51.3)
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Other:
- board size 295.9 x 105.4 mm -> 285 x 94.6 mm
